File: KiCAD/EnvironmentSensorTests.sch (KiCad schematic (older format))
At the start: 4 parts

Commit message: Correct schematic symbols and libraries.
Parts:
- removed A1: DHT-11_Board, symbol EnvironmentSensorTests-rescue:DHT-11_Board-Sensors-EnvironmentSensorTests-rescue
- removed A3: AdaFruit_ADT7410_Board, Sensors:AdaFruit_ADS7410_Board, symbol EnvironmentSensorTests-rescue:AdaFruit_ADT7410_Board-Sensors-EnvironmentSensorT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
- removed A4: SSD1306_128x64_OLED, Sensors:SSD1306_128x64_OLED_Display, symbol EnvironmentSensorTests-rescue:SSD1306_128x64_OLED-Sensors-EnvironmentSensorTest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
- added A?: DHT-11_Board, symbol zzzMyParts:DHT-11_Board
- added A?: AdaFruit_ADT7410_Board, symbol zzzMyParts:AdaFruit_ADT7410_Board
- added A?: SSD1306_128x64_OLED, symbol zzzMyParts:SSD1306_128x64_OLED
Connections:
- net GND: now also A?.1 (GND), A?.2 (GND), A?.3 (GND)
- net at A2.2 (3V3): now also A?.1 (VDD), A?.2 (VCC), A?.2 (VCC)
- net at A2.9 (SCL/15): now also A?.3 (SCL), A?.3 (SCL)
- net at A2.8 (SDA/A4): now also A?.4 (SDA), A?.4 (SDA)
- net at A2.20 (D2): now also A?.1 (DATA)
Changed lines of the file:
@@
 NoConn ~ 6850 4000
 NoConn ~ 6850 3800
-$Comp
-L EnvironmentSensorTests-rescue:SSD1306_128x64_OLED-Sensors-EnvironmentSensorTests-rescue A4
-U 1 1 5F49AE1E
-P 7850 3850
-F 0 "A4" H 7750 4100 50  0000 L CNN
-F 1 "SSD1306_128x64_OLED" H 8100 3450 50  0000 L CNN
-F 2 "Sensors:SSD1306_128x64_OLED_Display" H 7850 3850 50  0001 C CNN
-F 3 "" H 7850 3850 50  0001 C CNN
-	1    7850 3850
-	1    0    0    -1
-$EndComp
 Wire Wire Line
 	8000 3550 8000 3100
@@
 NoConn ~ 6100 3950
 NoConn ~ 6100 4050
-$Comp
-L EnvironmentSensorTests-rescue:AdaFruit_ADT7410_Board-Sensors-EnvironmentSensorTests-rescue A3
-U 1 1 5F4AF334
-P 6350 3900
-F 0 "A3" H 6350 4200 50  0000 C CNN
-F 1 "AdaFruit_ADT7410_Board" H 7050 4250 50  0000 C CNN
-F 2 "Sensors:AdaFruit_ADS7410_Board" H 6350 3900 50  0001 C CNN
-F 3 "" H 6350 3900 50  0001 C CNN
-	1    6350 3900
-	1    0    0    -1
-$EndComp
-$Comp
-L EnvironmentSensorTests-rescue:DHT-11_Board-Sensors-EnvironmentSensorTests-rescue A1
-U 1 1 5F4AA930
-P 3650 3800
-F 0 "A1" H 4050 4100 50  0000 L CNN
-F 1 "DHT-11_Board" H 3300 3500 50  0000 L CNN
-F 2 "" H 3650 3800 50  0001 C CNN
-F 3 "" H 3650 3800 50  0001 C CNN
-	1    3650 3800
-	-1   0    0    -1
-$EndComp
 Wire Wire Line
 	3800 3850 4000 3850
@@
 Wire Wire Line
 	4800 3100 6550 3100
+$Comp
+L zzzMyParts:DHT-11_Board A?
+U 1 1 5F4C3D8C
+P 3650 3800
+F 0 "A?" H 4178 3821 50  0000 L CNN
+F 1 "DHT-11_Board" H 4178 3730 50  0000 L CNN
+F 2 "" H 3650 3800 50  0001 C CNN
+F 3 "" H 3650 3800 50  0001 C CNN
+	1    3650 3800
+	-1   0    0    -1
+$EndComp
+$Comp
+L zzzMyParts:AdaFruit_ADT7410_Board A?
+U 1 1 5F4C550F
+P 6350 3900
+F 0 "A?" H 6525 4431 50  0000 C CNN
+F 1 "AdaFruit_ADT7410_Board" H 6525 4340 50  0000 C CNN
+F 2 "" H 6350 3900 50  0001 C CNN
+F 3 "" H 6350 3900 50  0001 C CNN
+	1    6350 3900
+	1    0    0    -1
+$EndComp
+$Comp
+L zzzMyParts:SSD1306_128x64_OLED A?
+U 1 1 5F4C654E
+P 7850 3850
+F 0 "A?" H 8278 3846 50  0000 L CNN
+F 1 "SSD1306_128x64_OLED" H 8278 3755 50  0000 L CNN
+F 2 "" H 7850 3850 50  0001 C CNN
+F 3 "" H 7850 3850 50  0001 C CNN
+	1    7850 3850
+	1    0    0    -1
+$EndComp
 $EndSCHEMATC
